Commit message: Fix demo Genesis launch and crane teleop

File: web/public/demo/crane/ship_crane.urdf (robot description, URDF)
Before this commit: robot ship_crane, 6 links, 5 joints
Links:
- link boom_link: mass 200433.6 -> 22.2
- link finger_link: mass 12.0 -> 0.013
- link gripper_palm: mass 100.0 -> 0.04
Joints:
- joint base_yaw: axis 0 1 0 -> (none); type continuous -> fixed
